File: design_files/ASD2841.sch (EAGLE design)
At the start: 15 parts, among them J1 DF12-32-DP, J2 DF12-32-DS, J3 SJ-3524-SMT-TR, U1 TS922IDT, U2 MCP4921T-E/MS

Commit message: update format
Parts:
- added R4: 1.00K, tinycircuits:AS-ITM-00003
- C7: value 1UF -> 1uF
- U1: value TS922IDT -> MCP4921T-E/MS; device tinycircuits:AS-ITM-00092 -> tinycircuits:AS-ITM-00091; VALUE TS922IDT -> MCP4921-E/MS
- U2: value MCP4921T-E/MS -> TS922IDT; device tinycircuits:AS-ITM-00091 -> tinycircuits:AS-ITM-00092; VALUE MCP4921-E/MS -> TS922IDT
- renumbered C12 to C7
Connections:
- net AD0: now also R4.1
- net GND: now also U1.LDAC, U1.VSS, U2.VCC-; no longer U1.VCC-, U2.LDAC, U2.VSS
- net IO2: now also U1.CS; no longer U2.CS
- net IO3: now also U1.SCK; no longer U2.SCK
- net IO4: now also U1.SDI; no longer U2.SDI
- net N$1: now also U2.2IN+, U2.IN1+; no longer U1.2IN+, U1.IN1+
- net N$2: now also U2.2IN-, U2.2OUT, U2.IN1-, U2.OUT1; no longer U1.2IN-, U1.2OUT, U1.IN1-, U1.OUT1
- net N$3: now also U1.VREF; no longer U2.VREF
- net N$4: now also U1.VOUT; no longer U2.VOUT
- net N$9: now also R4.2
- net VCC: now also U1.VDD, U2.VCC+; no longer U1.VCC+, U2.VDD
Other:
- note added: "5"
- note added: "Hand Populated: R1, J3, U1"
- note added: "Hand Soldered: -"
- note added: "Non Populated: -"
- note added: "Notes: -"
- note added: "Variant: Standard"
- note removed: "4"
